File: Breakout Board STM32L041x6 - TSSOP20/Breakout Board STM32L041x6 - TSSOP20.sch (KiCad schematic (older format))
At the start: 14 parts

Commit message: Update
Parts:
- removed Y?: Crystal_Small, symbol Device:Crystal_Small
- added D? (x2): LED_Small, symbol Device:LED_Small
- added D?: D_Schottky, symbol Device:D_Schottky
- added R? (x2): R_Small, symbol Device:R_Small
- added TP?: TestPoint swclk, symbol Connector:TestPoint
- added TP?: TestPoint swdio, symbol Connector:TestPoint
- added TP?: TestPoint vdd, symbol Connector:TestPoint
- added TP?: TestPoint gnd, symbol Connector:TestPoint
- added Y?: Crystal_GND2, symbol Device:Crystal_GND2
Connections:
- net labels added: led, swclk, swdio, vddext
- wire segments 54 -> 73
Other:
- moved on the sheet: C?, R?
