File: Breakout Board STM32L041x6 - TSSOP20/Breakout Board STM32L041x6 - TSSOP20.sch (KiCad schematic (older format))
At the start: 23 parts, among them J1 Conn_01x10, J2 Conn_01x10, SW1 SW_Push, U1 STM32L041x6-TSSOP20, Y1 Crystal_GND2

Commit message: Update
Parts:
- added C8: ???F, Diode_SMD:D_0805_2012Metric_Pad1.15x1.40mm_HandSolder, symbol Device:C_Small
- added R5, R6: R_Small, Resistor_SMD:R_0805_2012Metric_Pad1.15x1.40mm_HandSolder, symbol Device:R_Small
- added SW2: SW_Push, Breakout Board STM32L041x6 - TSSOP20:Tactile Switch TS-064 - Comet, symbol Switch:SW_Push
- J1, J2: footprint Connector_PinHeader_2.54mm:PinHeader_1x10_P2.54mm_Vertical -> Breakout Board STM32L041x6 - TSSOP20:PinHeader 1x10 P2.54mm Vertical
Connections:
- net labels added: button
- wire segments 73 -> 86
Changed lines of the file:
@@
 F 0 "J1" H 4170 2125 50  0000 C CNN
 F 1 "Conn_01x10" H 4170 2216 50  0000 C CNN
-F 2 "Connector_PinHeader_2.54mm:PinHeader_1x10_P2.54mm_Vertical" H 4250 2850 50  0001 C CNN
+F 2 "Breakout Board STM32L041x6 - TSSOP20:PinHeader 1x10 P2.54mm Vertical" H 4250 2850 50  0001 C CNN
 F 3 "~" H 4250 2850 50  0001 C CNN
 	1    4250 2850
@@
 F 0 "J2" H 6680 2742 50  0000 L CNN
 F 1 "Conn_01x10" H 6680 2651 50  0000 L CNN
-F 2 "Connector_PinHeader_2.54mm:PinHeader_1x10_P2.54mm_Vertical" H 6600 2750 50  0001 C CNN
+F 2 "Breakout Board STM32L041x6 - TSSOP20:PinHeader 1x10 P2.54mm Vertical" H 6600 2750 50  0001 C CNN
 F 3 "~" H 6600 2750 50  0001 C CNN
 	1    6600 2750
@@
 Text Label 6200 2350 0    50   ~ 0
 swclk
-Text Label 6200 2550 0    50   ~ 0
+Text Label 6200 3250 0    50   ~ 0
 led
 Wire Wire Line
@@
 NoConn ~ 4450 2450
 NoConn ~ 4450 2550
+Wire Wire Line
+	3600 3050 3550 3050
+Wire Wire Line
+	3550 3050 3550 3150
+$Comp
+L power:GND #PWR09
+U 1 1 5D2EEAAE
+P 3550 3150
+F 0 "#PWR09" H 3550 2900 50  0001 C CNN
+F 1 "GND" H 3555 2977 50  0000 C CNN
+F 2 "" H 3550 3150 50  0001 C CNN
+F 3 "" H 3550 3150 50  0001 C CNN
+	1    3550 3150
+	1    0    0    -1
+$EndComp
+Text Label 3600 3050 0    50   ~ 0
+gnd
+Wire Wire Line
+	5350 1900 5550 1900
+Text Label 5550 1900 0    50   ~ 0
+vdd
+Text Label 5350 1900 2    50   ~ 0
+vdda
+Text Label 4500 3250 0    50   ~ 0
+button
+$Comp
+L Switch:SW_Push SW2
+U 1 1 5D2F6274
+P 2550 2600
+F 0 "SW2" V 2600 2850 50  0000 R CNN
+F 1 "SW_Push" V 2700 3000 50  0000 R CNN
+F 2 "Breakout Board STM32L041x6 - TSSOP20:Tactile Switch TS-064 - Comet" H 2550 2800 50  0001 C CNN
+F 3 "" H 2550 2800 50  0001 C CNN
+	1    2550 2600
+	0    -1   -1   0
+$EndComp
+$Comp
+L power:GND #PWR08
+U 1 1 5D2F6280
+P 2750 2800
+F 0 "#PWR08" H 2750 2550 50  0001 C CNN
+F 1 "GND" H 2755 2627 50  0000 C CNN
+F 2 "" H 2750 2800 50  0001 C CNN
+F 3 "" H 2750 2800 50  0001 C CNN
+	1    2750 2800
+	1    0    0    -1
+$EndComp
+$Comp
+L Device:R_Small R5
+U 1 1 5D2F82A4
+P 2800 2400
+F 0 "R5" V 2600 2300 50  0000 L CNN
+F 1 "R_Small" V 2700 2200 50  0000 L CNN
+F 2 "Resistor_SMD:R_0805_2012Metric_Pad1.15x1.40mm_HandSolder" H 2800 2400 50  0001 C CNN
+F 3 "~" H 2800 2400 50  0001 C CNN
+	1    2800 2400
+	0    1    1    0
+$EndComp
+Text Label 3100 2400 0    50   ~ 0
+button
+$Comp
+L Device:R_Small R6
+U 1 1 5D305710
+P 2950 2200
+F 0 "R6" H 3009 2246 50  0000 L CNN
+F 1 "R_Small" H 3009 2155 50  0000 L CNN
+F 2 "Resistor_SMD:R_0805_2012Metric_Pad1.15x1.40mm_HandSolder" H 2950 2200 50  0001 C CNN
+F 3 "~" H 2950 2200 50  0001 C CNN
+	1    2950 2200
+	1    0    0    -1
+$EndComp
+Wire Wire Line
+	2950 2100 2950 2050
+Text Label 3000 2050 0    50   ~ 0
+vdd
+Wire Wire Line
+	3000 2050 2950 2050
+$Comp
+L Device:C_Small C8
+U 1 1 5D3109EF
+P 2950 2600
+F 0 "C8" H 3042 2646 50  0000 L CNN
+F 1 "???F" H 3042 2555 50  0000 L CNN
+F 2 "Diode_SMD:D_0805_2012Metric_Pad1.15x1.40mm_HandSolder" H 2950 2600 50  0001 C CNN
+F 3 "~" H 2950 2600 50  0001 C CNN
+	1    2950 2600
+	1    0    0    -1
+$EndComp
+Wire Wire Line
+	2950 2300 2950 2400
+Wire Wire Line
+	2550 2400 2700 2400
+Wire Wire Line
+	2900 2400 2950 2400
+Connection ~ 2950 2400
+Wire Wire Line
+	2550 2800 2750 2800
+Wire Wire Line
+	2950 2400 3100 2400
+Wire Wire Line
+	2950 2500 2950 2400
+Wire Wire Line
+	2950 2700 2950 2800
+Connection ~ 2750 2800
+Wire Wire Line
+	2750 2800 2950 2800
 $EndSCHEMATC

Commit message: Update
Parts:
- C8: value ???F -> 100nF
- D1: value LED_Small -> ledvdd
- D2: value LED_Small -> led
- D3: value D_Schottky -> Dvddext
- R1: value R_Small -> 100k
- R2, R3: value R_Small -> Rled
- R4: value R_Small -> Rxtal
- R5: value R_Small -> 1k
- R6: value R_Small -> 10k
- SW1: value SW_Push -> user button
- SW2: value SW_Push -> reset switch
Connections:
- net labels added: key
- wire segments 86 -> 89
- no-connect marks 2 -> 1
Changed lines of the file:
@@
 U 1 1 5D2D186C
 P 4250 2850
-F 0 "J1" H 4170 2125 50  0000 C CNN
-F 1 "Conn_01x10" H 4170 2216 50  0000 C CNN
+F 0 "J1" H 4350 2150 50  0000 C CNN
+F 1 "Conn_01x10" H 4450 2250 50  0000 C CNN
 F 2 "Breakout Board STM32L041x6 - TSSOP20:PinHeader 1x10 P2.54mm Vertical" H 4250 2850 50  0001 C CNN
 F 3 "~" H 4250 2850 50  0001 C CNN
@@
 Wire Wire Line
 	4750 2350 4450 2350
-Text Label 4450 2350 0    50   ~ 0
+Text Label 4550 2350 1    50   ~ 0
 boot
 Wire Wire Line
@@
 P 3750 3800
 F 0 "R1" H 3809 3846 50  0000 L CNN
-F 1 "R_Small" H 3809 3755 50  0000 L CNN
+F 1 "100k" H 3809 3755 50  0000 L CNN
 F 2 "Resistor_SMD:R_0805_2012Metric_Pad1.15x1.40mm_HandSolder" H 3750 3800 50  0001 C CNN
 F 3 "~" H 3750 3800 50  0001 C CNN
@@
 Text Label 6200 2850 0    50   ~ 0
 gnd
-Text Label 4750 2450 2    50   ~ 0
+Text Label 4650 2450 1    50   ~ 0
 osc32in
-Text Label 4750 2550 2    50   ~ 0
+Text Label 4750 2550 1    50   ~ 0
 osc32out
 Text Label 6200 2750 0    50   ~ 0
@@
 P 7850 3700
 F 0 "R4" H 7909 3746 50  0000 L CNN
-F 1 "R_Small" H 7909 3655 50  0000 L CNN
+F 1 "Rxtal" H 7909 3655 50  0000 L CNN
 F 2 "Resistor_SMD:R_0805_2012Metric_Pad1.15x1.40mm_HandSolder" H 7850 3700 50  0001 C CNN
 F 3 "~" H 7850 3700 50  0001 C CNN
@@
 P 2800 3800
 F 0 "SW1" V 2850 4050 50  0000 R CNN
-F 1 "SW_Push" V 2950 4200 50  0000 R CNN
+F 1 "user button" V 2950 4200 50  0000 R CNN
 F 2 "Breakout Board STM32L041x6 - TSSOP20:Tactile Switch TS-064 - Comet" H 2800 4000 50  0001 C CNN
 F 3 "" H 2800 4000 50  0001 C CNN
@@
 P 6000 3750
 F 0 "D1" V 6046 3682 50  0000 R CNN
-F 1 "LED_Small" V 5955 3682 50  0000 R CNN
+F 1 "ledvdd" V 5955 3682 50  0000 R CNN
 F 2 "LED_SMD:LED_1206_3216Metric_Pad1.42x1.75mm_HandSolder" V 6000 3750 50  0001 C CNN
 F 3 "~" V 6000 3750 50  0001 C CNN
@@
 P 6000 4000
 F 0 "R2" H 6059 4046 50  0000 L CNN
-F 1 "R_Small" H 6059 3955 50  0000 L CNN
+F 1 "Rled" H 6059 3955 50  0000 L CNN
 F 2 "Resistor_SMD:R_0805_2012Metric_Pad1.15x1.40mm_HandSolder" H 6000 4000 50  0001 C CNN
 F 3 "~" H 6000 4000 50  0001 C CNN
@@
 P 6400 3750
 F 0 "D2" V 6446 3682 50  0000 R CNN
-F 1 "LED_Small" V 6355 3682 50  0000 R CNN
+F 1 "led" V 6355 3682 50  0000 R CNN
 F 2 "LED_SMD:LED_1206_3216Metric_Pad1.42x1.75mm_HandSolder" V 6400 3750 50  0001 C CNN
 F 3 "~" V 6400 3750 50  0001 C CNN
@@
 P 6400 4000
 F 0 "R3" H 6459 4046 50  0000 L CNN
-F 1 "R_Small" H 6459 3955 50  0000 L CNN
+F 1 "Rled" H 6459 3955 50  0000 L CNN
 F 2 "Resistor_SMD:R_0805_2012Metric_Pad1.15x1.40mm_HandSolder" H 6400 4000 50  0001 C CNN
 F 3 "~" H 6400 4000 50  0001 C CNN
@@
 P 8450 2700
 F 0 "D3" V 8496 2621 50  0000 R CNN
-F 1 "D_Schottky" V 8405 2621 50  0000 R CNN
+F 1 "Dvddext" V 8405 2621 50  0000 R CNN
 F 2 "Diode_SMD:D_SOD-123" H 8450 2700 50  0001 C CNN
 F 3 "~" H 8450 2700 50  0001 C CNN
@@
 Wire Wire Line
 	4750 2550 4550 2550
-NoConn ~ 4450 2450
-NoConn ~ 4450 2550
 Wire Wire Line
 	3600 3050 3550 3050
@@
 P 2550 2600
 F 0 "SW2" V 2600 2850 50  0000 R CNN
-F 1 "SW_Push" V 2700 3000 50  0000 R CNN
+F 1 "reset switch" V 2700 3000 50  0000 R CNN
 F 2 "Breakout Board STM32L041x6 - TSSOP20:Tactile Switch TS-064 - Comet" H 2550 2800 50  0001 C CNN
 F 3 "" H 2550 2800 50  0001 C CNN
@@
 P 2800 2400
 F 0 "R5" V 2600 2300 50  0000 L CNN
-F 1 "R_Small" V 2700 2200 50  0000 L CNN
+F 1 "1k" V 2700 2200 50  0000 L CNN
 F 2 "Resistor_SMD:R_0805_2012Metric_Pad1.15x1.40mm_HandSolder" H 2800 2400 50  0001 C CNN
 F 3 "~" H 2800 2400 50  0001 C CNN
@@
 P 2950 2200
 F 0 "R6" H 3009 2246 50  0000 L CNN
-F 1 "R_Small" H 3009 2155 50  0000 L CNN
+F 1 "10k" H 3009 2155 50  0000 L CNN
 F 2 "Resistor_SMD:R_0805_2012Metric_Pad1.15x1.40mm_HandSolder" H 2950 2200 50  0001 C CNN
 F 3 "~" H 2950 2200 50  0001 C CNN
@@
 P 2950 2600
 F 0 "C8" H 3042 2646 50  0000 L CNN
-F 1 "???F" H 3042 2555 50  0000 L CNN
+F 1 "100nF" H 3042 2555 50  0000 L CNN
 F 2 "Diode_SMD:D_0805_2012Metric_Pad1.15x1.40mm_HandSolder" H 2950 2600 50  0001 C CNN
 F 3 "~" H 2950 2600 50  0001 C CNN
@@
 Wire Wire Line
 	2750 2800 2950 2800
+Wire Wire Line
+	4450 2450 4500 2450
+Text Label 4450 2450 1    50   ~ 0
+gnd
+Wire Wire Line
+	4450 2550 4500 2550
+Text Label 4500 2550 1    50   ~ 0
+key
+Wire Wire Line
+	4350 1950 4400 1950
+Text Label 4350 1950 2    50   ~ 0
+key
+NoConn ~ 4400 1950
 $EndSCHEMATC

Commit message: Update
Parts:
- removed U1: STM32L041x6-TSSOP20, Breakout Board STM32L041x6 - TSSOP20:STM32L041x6 - TSSOP20, symbol STM32L041x6~-~TSSOP20:STM32L041x6-TSSOP20
- added U1: STM32L041F6P7, Breakout Board STM32L041x6 - TSSOP20:STM32L041x6 - TSSOP20, symbol Breakout-Board-STM32L041x6---TSSOP20-rescue:STM32L041x6-TSSOP20-STM32L041x6_-_T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
- D1: value ledvdd -> led power
- D2: value led -> user led
- SW1: value user button -> reset switch
- SW2: value reset switch -> user switch
- TP1: value TestPoint swclk -> swdio
- TP2: value TestPoint swdio -> swclk
- TP3: value TestPoint vdd -> vddext
- TP4: value TestPoint gnd -> gnd
- Y1: value Crystal_GND2 -> Crystal 32768
Connections:
- net labels added: switch
- net labels removed: button
- wire segments 89 -> 95
Other:
- note added: "Debug connection (SWD - serial wire debug)"
- note added: "Indication/user input"
- note added: "Microcontroller"
- note added: "System setup - reset, clock, boot configuratin"
- moved on the sheet: C1, C2, C3, C4, C5, C6, C7, C8, D1, D2, D3, J1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

Commit message: Update
Connections:
- net pa3: now reaches J1.2 (Pin_2), U1.9 (PA3)
- net pa2: now reaches J1.3 (Pin_3), U1.8 (PA2)
- net pa1: now reaches J1.4 (Pin_4), U1.7 (PA1)
- net pa0: now reaches J1.5 (Pin_5), U1.6 (PA0)
- net pa10: now reaches J2.3 (Pin_3), U1.18 (PA10)
- net pa9: now reaches J2.4 (Pin_4), U1.17 (PA9)
- net pb1: now reaches J2.7 (Pin_7), U1.14 (PB1)
- net pa7: now reaches J2.8 (Pin_8), U1.13 (PA7)
- net pa6: now reaches J2.9 (Pin_9), U1.12 (PA6)
Changed lines of the file:
@@
 Wire Wire Line
 	4900 2900 4950 2900
+Text Label 4800 3700 0    50   ~ 0
+pa0
+Text Label 4800 3800 0    50   ~ 0
+pa1
+Text Label 4800 3900 0    50   ~ 0
+pa2
+Text Label 4800 4000 0    50   ~ 0
+pa3
+Text Label 6500 4000 0    50   ~ 0
+pa6
+Text Label 6500 3900 0    50   ~ 0
+pa7
+Text Label 6500 3800 0    50   ~ 0
+pb1
+Text Label 6500 3500 0    50   ~ 0
+pa9
+Text Label 6500 3400 0    50   ~ 0
+pa10
 $EndSCHEMATC

Commit message: Update
Parts:
- D1: value led power -> led - power
Changed lines of the file:
@@
 P 1750 3300
 F 0 "D1" V 1700 3250 50  0000 R CNN
-F 1 "led power" V 1850 3250 50  0000 R CNN
+F 1 "led - power" V 2000 3400 50  0000 R CNN
 F 2 "LED_SMD:LED_1206_3216Metric_Pad1.42x1.75mm_HandSolder" V 1750 3300 50  0001 C CNN
 F 3 "~" V 1750 3300 50  0001 C CNN

Commit message: Update
Parts:
- added TP5: x1, Breakout Board STM32L041x6 - TSSOP20:TestPoint 2.54mm round, symbol Connector:TestPoint
- added TP6: x2, Breakout Board STM32L041x6 - TSSOP20:TestPoint 2.54mm round, symbol Connector:TestPoint
- added TP7: x3, Breakout Board STM32L041x6 - TSSOP20:TestPoint 2.54mm round, symbol Connector:TestPoint
- added TP8: x4, Breakout Board STM32L041x6 - TSSOP20:TestPoint 2.54mm round, symbol Connector:TestPoint
- D2: value user led -> goldstar
- SW2: value user switch -> ibm m
Connections:
- net led renamed goldstar
- net switch renamed ibm-m
- no-connect marks 1 -> 5
Other:
- note added: "Bypass shaft"
Changed lines of the file:
@@
 Text Label 6500 3200 0    50   ~ 0
 swclk
-Text Label 6500 4100 0    50   ~ 0
-led
+Text Label 6400 4100 0    50   ~ 0
+goldstar
 Wire Wire Line
 	1800 3150 1750 3150
@@
 P 2150 3300
 F 0 "D2" V 2196 3232 50  0000 R CNN
-F 1 "user led" V 2105 3232 50  0000 R CNN
+F 1 "goldstar" V 2105 3232 50  0000 R CNN
 F 2 "LED_SMD:LED_1206_3216Metric_Pad1.42x1.75mm_HandSolder" V 2150 3300 50  0001 C CNN
 F 3 "~" V 2150 3300 50  0001 C CNN
@@
 vdd
 Text Label 2200 3150 0    50   ~ 0
-led
+goldstar
 $Comp
 L Connector:TestPoint TP1
@@
 Text Label 6450 4800 2    50   ~ 0
 vdda
-Text Label 4800 4100 0    50   ~ 0
-switch
+Text Label 4750 4100 0    50   ~ 0
+ibm-m
 $Comp
 L Switch:SW_Push SW2
@@
 P 2750 3650
 F 0 "SW2" V 2800 3900 50  0000 R CNN
-F 1 "user switch" V 2950 4100 50  0000 R CNN
+F 1 "ibm m" V 2900 3950 50  0000 R CNN
 F 2 "Breakout Board STM32L041x6 - TSSOP20:Tactile Switch TS-064 - Comet" H 2750 3850 50  0001 C CNN
 F 3 "" H 2750 3850 50  0001 C CNN
@@
 $EndComp
 Text Label 3300 3450 0    50   ~ 0
-switch
+ibm-m
 $Comp
 L Device:R_Small R6
@@
 Text Label 6500 3400 0    50   ~ 0
 pa10
+$Comp
+L Connector:TestPoint TP5
+U 1 1 5D2F9664
+P 8550 1750
+F 0 "TP5" V 8600 1750 50  0000 C CNN
+F 1 "x1" V 8550 2050 50  0000 C CNN
+F 2 "Breakout Board STM32L041x6 - TSSOP20:TestPoint 2.54mm round" H 8750 1750 50  0001 C CNN
+F 3 "~" H 8750 1750 50  0001 C CNN
+	1    8550 1750
+	0    -1   -1   0
+$EndComp
+$Comp
+L Connector:TestPoint TP6
+U 1 1 5D2F966A
+P 8550 1850
+F 0 "TP6" V 8600 1850 50  0000 C CNN
+F 1 "x2" V 8550 2150 50  0000 C CNN
+F 2 "Breakout Board STM32L041x6 - TSSOP20:TestPoint 2.54mm round" H 8750 1850 50  0001 C CNN
+F 3 "~" H 8750 1850 50  0001 C CNN
+	1    8550 1850
+	0    -1   -1   0
+$EndComp
+$Comp
+L Connector:TestPoint TP7
+U 1 1 5D2FC439
+P 8550 1950
+F 0 "TP7" V 8600 1950 50  0000 C CNN
+F 1 "x3" V 8550 2250 50  0000 C CNN
+F 2 "Breakout Board STM32L041x6 - TSSOP20:TestPoint 2.54mm round" H 8750 1950 50  0001 C CNN
+F 3 "~" H 8750 1950 50  0001 C CNN
+	1    8550 1950
+	0    -1   -1   0
+$EndComp
+$Comp
+L Connector:TestPoint TP8
+U 1 1 5D2FC43F
+P 8550 2050
+F 0 "TP8" V 8600 2050 50  0000 C CNN
+F 1 "x4" V 8550 2350 50  0000 C CNN
+F 2 "Breakout Board STM32L041x6 - TSSOP20:TestPoint 2.54mm round" H 8750 2050 50  0001 C CNN
+F 3 "~" H 8750 2050 50  0001 C CNN
+	1    8550 2050
+	0    -1   -1   0
+$EndComp
+Text Notes 8200 1600 0    50   ~ 0
+Bypass shaft
+Wire Notes Line
+	8150 1500 8750 1500
+Wire Notes Line
+	8750 1500 8750 2100
+Wire Notes Line
+	8750 2100 8150 2100
+Wire Notes Line
+	8150 2100 8150 1500
+NoConn ~ 8550 1750
+NoConn ~ 8550 1850
+NoConn ~ 8550 1950
+NoConn ~ 8550 2050
 $EndSCHEMATC

Commit message: Update
Changed lines of the file:
@@
 Wire Notes Line
 	8150 2100 8150 1500
-NoConn ~ 8550 1750
-NoConn ~ 8550 1850
-NoConn ~ 8550 1950
-NoConn ~ 8550 2050
+NoConn ~ 8600 1750
+NoConn ~ 8600 1850
+NoConn ~ 8600 1950
+NoConn ~ 8600 2050
+Wire Wire Line
+	8550 2050 8600 2050
+Wire Wire Line
+	8600 1950 8550 1950
+Wire Wire Line
+	8600 1850 8550 1850
+Wire Wire Line
+	8600 1750 8550 1750
 $EndSCHEMATC

Commit message: Update
Parts:
- D2: value goldstar -> LED
- SW2: value ibm m -> switch
Connections:
- net goldstar renamed led
- net ibm-m renamed switch
Changed lines of the file:
@@
 swclk
 Text Label 6400 4100 0    50   ~ 0
-goldstar
+led
 Wire Wire Line
 	1800 3150 1750 3150
@@
 P 2150 3300
 F 0 "D2" V 2196 3232 50  0000 R CNN
-F 1 "goldstar" V 2105 3232 50  0000 R CNN
+F 1 "LED" V 2105 3232 50  0000 R CNN
 F 2 "LED_SMD:LED_1206_3216Metric_Pad1.42x1.75mm_HandSolder" V 2150 3300 50  0001 C CNN
 F 3 "~" V 2150 3300 50  0001 C CNN
@@
 vdd
 Text Label 2200 3150 0    50   ~ 0
-goldstar
+led
 $Comp
 L Connector:TestPoint TP1
@@
 vdda
 Text Label 4750 4100 0    50   ~ 0
-ibm-m
+switch
 $Comp
 L Switch:SW_Push SW2
@@
 P 2750 3650
 F 0 "SW2" V 2800 3900 50  0000 R CNN
-F 1 "ibm m" V 2900 3950 50  0000 R CNN
+F 1 "switch" V 2900 3950 50  0000 R CNN
 F 2 "Breakout Board STM32L041x6 - TSSOP20:Tactile Switch TS-064 - Comet" H 2750 3850 50  0001 C CNN
 F 3 "" H 2750 3850 50  0001 C CNN
@@
 $EndComp
 Text Label 3300 3450 0    50   ~ 0
-ibm-m
+switch
 $Comp
 L Device:R_Small R6
