File: Breakout Board STM32L041x6 - TSSOP20/Breakout Board STM32L041x6 - TSSOP20.kicad_pcb (KiCad board)
At the start: 2 copper layers, 35.6 x 33 mm, 27 parts, among them J1 Conn_01x10, J2 Conn_01x10, SW1 SW_Push, SW2 SW_Push, U1 STM32L041x6-TSSOP20, Y1 Crystal_GND2

Commit message: Update
Parts:
- moved C7 5.87 mm to (118.8, 83.0), turned to 270 degrees
- moved D3 1.90 mm to (132.5, 85.8)
Routing:
- net GND: track 37.3 -> 41.0 mm
- net /osc32out: track 1.68 -> 3.72 mm, vias 0 -> 1
- net Net-(C7-Pad1): track 6.16 -> 7.45 mm
- net /osc32in: track 5.40 -> 5.60 mm, vias 0 -> 1
Changed lines of the file:
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@@
     (thickness 1.6)
     (drawings 10)
-    (tracks 22)
+    (tracks 31)
     (zones 0)
     (modules 27)
@@
   )
   (module Diode_SMD:D_0805_2012Metric_Pad1.15x1.40mm_HandSolder (layer B.Cu)
-    (at 124.275 85)
+    (at 118.75 83.025 270)
     (descr "Diode SMD 0805 (2012 Metric), square (rectangular) end terminal, IPC_7351 nominal, (Body size source: https://docs.google.com/spreadsheets/d/1BsfQQcO9C6DZCsRaXUlFlo91Tg2WpOkGARC1WS5S8t0/edit?usp=sharing), generated with kicad-footprint-generator")
     (tags "diode handsolder")
     (attr smd)
-    (fp_text reference C7 (at 0 1.65) (layer B.SilkS)
-      (effects (font (size 1 1) (thickness 0.15)) (justify mirror))
-    )
-    (fp_text value 6pF (at 0 -1.65) (layer B.Fab)
-      (effects (font (size 1 1) (thickness 0.15)) (justify mirror))
-    )
-    (fp_text user %R (at 0 0) (layer B.Fab)
+    (fp_text reference C7 (at 0 1.65 270) (layer B.SilkS)
+      (effects (font (size 1 1) (thickness 0.15)) (justify mirror))
+    )
+    (fp_text value 6pF (at 0 -1.65 270) (layer B.Fab)
+      (effects (font (size 1 1) (thickness 0.15)) (justify mirror))
+    )
+    (fp_text user %R (at 0 0 270) (layer B.Fab)
       (effects (font (size 0.5 0.5) (thickness 0.08)) (justify mirror))
     )
@@
     (fp_line (start -0.7 0.6) (end -1 0.3) (layer B.Fab) (width 0.1))
     (fp_line (start 1 0.6) (end -0.7 0.6) (layer B.Fab) (width 0.1))
-    (pad 2 smd roundrect (at 1.025 0) (size 1.15 1.4) (layers B.Cu B.Paste B.Mask) (roundrect_rratio 0.217391)
-      (net 2 GND))
-    (pad 1 smd roundrect (at -1.025 0) (size 1.15 1.4) (layers B.Cu B.Paste B.Mask) (roundrect_rratio 0.217391)
+    (pad 2 smd roundrect (at 1.025 0 270) (size 1.15 1.4) (layers B.Cu B.Paste B.Mask) (roundrect_rratio 0.217391)
+      (net 2 GND))
+    (pad 1 smd roundrect (at -1.025 0 270) (size 1.15 1.4) (layers B.Cu B.Paste B.Mask) (roundrect_rratio 0.217391)
       (net 5 "Net-(C7-Pad1)"))
     (model ${KISYS3DMOD}/Diode_SMD.3dshapes/D_0805_2012Metric.wrl
@@
   )
   (module Diode_SMD:D_SOD-123 (layer B.Cu)
-    (at 134.25 86.6 270)
+    (at 132.5 85.85 270)
     (descr SOD-123)
     (tags SOD-123)
@@
   (segment (start 130.7 77.7) (end 132.25 79.25) (width 0.25) (layer B.Cu) (net 2))
   (segment (start 121 77.7) (end 130.7 77.7) (width 0.25) (layer B.Cu) (net 2) (status 10))
-  (segment (start 129.5 85) (end 125.3 85) (width 0.25) (layer B.Cu) (net 2) (status 20))
-  (segment (start 132.25 82.25) (end 129.5 85) (width 0.25) (layer B.Cu) (net 2))
-  (segment (start 132.25 80.75) (end 132.25 82.25) (width 0.25) (layer B.Cu) (net 2) (status 10))
-  (segment (start 119.25 83.9589) (end 119.25 81.25) (width 0.25) (layer B.Cu) (net 2))
-  (segment (start 121.36611 86.07501) (end 119.25 83.9589) (width 0.25) (layer B.Cu) (net 2))
-  (segment (start 125.3 85) (end 124.22499 86.07501) (width 0.25) (layer B.Cu) (net 2) (status 10))
-  (segment (start 124.22499 86.07501) (end 121.36611 86.07501) (width 0.25) (layer B.Cu) (net 2))
-  (segment (start 119.25 79.45) (end 121 77.7) (width 0.25) (layer B.Cu) (net 2) (status 20))
-  (segment (start 119.25 81.25) (end 119.25 79.45) (width 0.25) (layer B.Cu) (net 2))
-  (segment (start 121.548837 80.298837) (end 121 79.75) (width 0.25) (layer B.Cu) (net 4) (status 30))
-  (segment (start 122.567444 80.298837) (end 121.548837 80.298837) (width 0.25) (layer B.Cu) (net 4) (status 20))
+  (segment (start 119.373372 84.673372) (end 118.75 84.05) (width 0.25) (layer B.Cu) (net 2))
+  (segment (start 119.70001 85.00001) (end 119.373372 84.673372) (width 0.25) (layer B.Cu) (net 2))
+  (segment (start 129.49999 85.00001) (end 119.70001 85.00001) (width 0.25) (layer B.Cu) (net 2))
+  (segment (start 132.25 82.25) (end 129.49999 85.00001) (width 0.25) (layer B.Cu) (net 2))
+  (segment (start 132.25 80.75) (end 132.25 82.25) (width 0.25) (layer B.Cu) (net 2))
+  (segment (start 116.8 82.1) (end 116.8 78.25) (width 0.25) (layer B.Cu) (net 2))
+  (segment (start 118.75 84.05) (end 116.8 82.1) (width 0.25) (layer B.Cu) (net 2))
+  (segment (start 120.45 78.25) (end 121 77.7) (width 0.25) (layer B.Cu) (net 2))
+  (segment (start 116.8 78.25) (end 120.45 78.25) (width 0.25) (layer B.Cu) (net 2))
   (segment (start 124.25 79.75) (end 124.5 79.5) (width 0.25) (layer B.Cu) (net 4) (status 30))
-  (segment (start 121 79.75) (end 124.25 79.75) (width 0.25) (layer B.Cu) (net 4) (status 30))
-  (segment (start 122.3 84.05) (end 123.25 85) (width 0.25) (layer B.Cu) (net 5) (status 20))
-  (segment (start 121 84.05) (end 122.3 84.05) (width 0.25) (layer B.Cu) (net 5) (status 10))
-  (segment (start 124.5 83.75) (end 124.5 82) (width 0.25) (layer B.Cu) (net 5) (status 20))
-  (segment (start 123.25 85) (end 124.5 83.75) (width 0.25) (layer B.Cu) (net 5) (status 10))
+  (via (at 122.572559 79.743691) (size 0.8) (drill 0.4) (layers F.Cu B.Cu) (net 4))
+  (segment (start 122.572559 80.252441) (end 122.572559 79.743691) (width 0.25) (layer F.Cu) (net 4))
+  (segment (start 122.175 80.65) (end 122.572559 80.252441) (width 0.25) (layer F.Cu) (net 4))
+  (segment (start 121.25 80.65) (end 122.175 80.65) (width 0.25) (layer F.Cu) (net 4))
+  (segment (start 121 79.75) (end 122.572559 79.743691) (width 0.25) (layer B.Cu) (net 4))
+  (segment (start 122.572559 79.743691) (end 124.25 79.75) (width 0.25) (layer B.Cu) (net 4))
+  (segment (start 123.75 82) (end 124.5 82) (width 0.25) (layer B.Cu) (net 5))
+  (segment (start 122.323372 83.426628) (end 123.75 82) (width 0.25) (layer B.Cu) (net 5))
+  (segment (start 121.623372 83.426628) (end 122.323372 83.426628) (width 0.25) (layer B.Cu) (net 5))
+  (segment (start 121 84.05) (end 121.623372 83.426628) (width 0.25) (layer B.Cu) (net 5))
+  (segment (start 120.8 84.05) (end 121 84.05) (width 0.25) (layer B.Cu) (net 5))
+  (segment (start 118.75 82) (end 120.8 84.05) (width 0.25) (layer B.Cu) (net 5))
   (segment (start 121.25 81.75) (end 121 82) (width 0.25) (layer B.Cu) (net 23) (status 30))
-  (segment (start 122.575002 81.75) (end 121.25 81.75) (width 0.25) (layer B.Cu) (net 23) (status 20))
+  (via (at 122.575002 82) (size 0.8) (drill 0.4) (layers F.Cu B.Cu) (net 23))
+  (segment (start 122.575002 81.700002) (end 122.575002 82) (width 0.25) (layer F.Cu) (net 23))
+  (segment (start 121.25 81.3) (end 122.175 81.3) (width 0.25) (layer F.Cu) (net 23))
+  (segment (start 122.175 81.3) (end 122.575002 81.700002) (width 0.25) (layer F.Cu) (net 23))
+  (segment (start 122.575002 82) (end 121 82) (width 0.25) (layer B.Cu) (net 23))
 )

Commit message: Update
Parts:
- C8: value ???F -> 100nF
- D1: value LED_Small -> ledvdd
- D2: value LED_Small -> led
- D3: value D_Schottky -> Dvddext
- R1: value R_Small -> 100k
- R2, R3: value R_Small -> Rled
- R4: value R_Small -> Rxtal
- R5: value R_Small -> 1k
- R6: value R_Small -> 10k
- SW1: value SW_Push -> user button
- SW2: value SW_Push -> reset switch
- moved D3 0.71 mm to (133.0, 86.3)
Connections:
- net Net-(J1-Pad8) renamed /key
- J1 pad 9: Net-(J1-Pad9) -> GND

Commit message: Update
Parts:
- D1: value ledvdd -> led power
- D2: value led -> user led
- SW1: value user button -> reset switch
- SW2: value reset switch -> user switch
- TP1: value TestPoint swclk -> swdio
- TP2: value TestPoint swdio -> swclk
- TP3: value TestPoint vdd -> vddext
- TP4: value TestPoint gnd -> gnd
- U1: value STM32L041x6-TSSOP20 -> STM32L041F6P7
- Y1: value Crystal_GND2 -> Crystal 32768
Connections:
- net /button renamed /switch

Commit message: Update
Parts:
- moved C2 12.5 mm to (128.4, 86.3)
- moved C3 12.5 mm to (130.4, 86.3)
- moved C6 12.5 mm to (132.4, 83.8)
- moved C8 12.5 mm to (126.4, 100.3)
- moved D3 12.5 mm to (144.4, 91.4)
- moved C4 12.5 mm to (143.9, 88.1)
- moved C5 12.5 mm to (141.7, 88.1)
- moved C7 12.5 mm to (130.2, 88.1)
- moved D1 12.5 mm to (126.2, 86.8)
- moved D2 12.5 mm to (141.7, 95.3)
- moved J2 12.5 mm to (148.6, 76.2)
- moved R3 12.5 mm to (141.7, 100.1)
- moved R4 12.5 mm to (132.4, 88.1)
- moved R5 12.5 mm to (126.4, 100.4)
- moved R6 12.5 mm to (126.4, 96.4)
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Connections:
- net Net-(J1-Pad2) renamed /pa3
- net Net-(J1-Pad3) renamed /pa2
- net Net-(J1-Pad4) renamed /pa1
- net Net-(J1-Pad5) renamed /pa0
- net Net-(J2-Pad3) renamed /pa10
- net Net-(J2-Pad4) renamed /pa9
- net Net-(J2-Pad7) renamed /pb1
- net Net-(J2-Pad8) renamed /pa7
- net Net-(J2-Pad9) renamed /pa6
Other:
- board text added: "AND"
- board text added: "NC/ key"
- board text added: "boot0"
- board text added: "gnd"
- board text added: "nrst"
- board text added: "pa0"
- board text added: "pa1"
- board text added: "pa10"
- board text added: "pa13 swdio"
- board text added: "pa14 swclk"
- board text added: "pa2"
- board text added: "pa3"
- board text added: "pa4"
- board text added: "pa5"
- board text added: "pa6"
- board text added: "pa7"
- board text added: "pa9"
- board text added: "pb1"
- board text added: "user led"
- board text added: "user switch"
- board text added: "vdd"

Commit message: Update
Parts:
- D1: value led power -> led - power
- moved TP3 13.4 mm to (141.0, 86.4)
- moved C1 13.3 mm to (123.4, 70.6)
- moved C2 13.3 mm to (124.6, 73.6)
- moved C3 13.3 mm to (126.6, 73.6)
- moved C4 13.3 mm to (140.1, 75.4)
- moved C5 13.3 mm to (137.9, 75.4)
- moved C6 13.3 mm to (128.6, 71.1)
- moved C7 13.3 mm to (126.4, 75.4)
- moved C8 13.3 mm to (122.6, 87.6)
- moved D1 13.3 mm to (122.4, 74.1)
- moved D2 13.3 mm to (137.9, 82.6)
- moved D3 13.3 mm to (140.6, 78.7)
- moved J1 13.3 mm to (119.4, 86.4)
- moved J2 13.3 mm to (144.8, 63.5)
- moved R2 13.3 mm to (123.4, 70.6)
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
Commit message: Update
Parts:
- added ?: , , F.Cu at (152.4, 59.1)
- added ?: , , F.Cu at (7.62, 17.8)
- added ?: , , F.Cu at (136.5, 81.9)
- added ?: , , F.Cu at (19.7, 0.00)
- added TP5: x1, Breakout Board STM32L041x6 - TSSOP20:TestPoint 2.54mm round, F.Cu at (116.8, 61.0)
- added TP6: x2, Breakout Board STM32L041x6 - TSSOP20:TestPoint 2.54mm round, F.Cu at (147.3, 61.0)
- added TP7: x3, Breakout Board STM32L041x6 - TSSOP20:TestPoint 2.54mm round, F.Cu at (116.8, 88.9)
- added TP8: x4, Breakout Board STM32L041x6 - TSSOP20:TestPoint 2.54mm round, F.Cu at (147.3, 88.9)
- D2: value user led -> goldstar
- SW2: value user switch -> ibm m
Connections:
- net /led renamed /goldstar
- net /switch renamed /ibm-m
Other:
- board text added: "a4& IBMM"
- board text added: "a5& STAR"
- board text added: "x1"
- board text added: "x2"
- board text added: "x3"
- board text added: "x4"
- board text removed: "AND"
- board text removed: "pa4"
- board text removed: "pa5"
- board text removed: "user led"
- board text removed: "user switch"

Commit message: Add insignia
Other:
- board text added: "ЕС1832 17072019а0"
- board text added: "ЕС1832 Терминален блок Проектирано и изработено в Република България"
Changed lines of the file:
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@@
   (general
     (thickness 1.6)
-    (drawings 90)
+    (drawings 92)
     (tracks 31)
     (zones 0)
@@
       (effects (font (size 1.27 1.27) (thickness 0.15)))
     )
-    (fp_text user x2 (at 0 20.32) (layer F.Fab)
+    (fp_text user x2 (at -5.08 1.905) (layer F.Fab) hide
       (effects (font (size 1 1) (thickness 0.15)))
     )
@@
     (tags "diode handsolder")
     (attr smd)
-    (fp_text reference C7 (at 3.975 0.25) (layer B.SilkS)
-      (effects (font (size 0.8 0.8) (thickness 0.15)) (justify mirror))
-    )
-    (fp_text value 6pF (at 2.725 0.5) (layer B.SilkS)
+    (fp_text reference C7 (at 0.16 2.545) (layer B.SilkS)
+      (effects (font (size 0.8 0.8) (thickness 0.15)) (justify mirror))
+    )
+    (fp_text value 6pF (at -1.11 2.545) (layer B.SilkS)
       (effects (font (size 0.8 0.8) (thickness 0.15)) (justify mirror))
     )
@@
     (tags SOD-123)
     (attr smd)
-    (fp_text reference D3 (at 0.15 1.75 270) (layer B.SilkS)
-      (effects (font (size 0.8 0.8) (thickness 0.15)) (justify mirror))
-    )
-    (fp_text value Dvddext (at 0 -2.1 270) (layer B.SilkS)
+    (fp_text reference D3 (at 3.185 -2.255 270) (layer B.SilkS)
+      (effects (font (size 0.8 0.8) (thickness 0.15)) (justify mirror))
+    )
+    (fp_text value Dvddext (at -0.625 -2.1 270) (layer B.SilkS)
       (effects (font (size 0.8 0.8) (thickness 0.15)) (justify mirror))
     )
@@
     (tags "resistor handsolder")
     (attr smd)
-    (fp_text reference R4 (at 3.975 0) (layer B.SilkS)
-      (effects (font (size 0.8 0.8) (thickness 0.15)) (justify mirror))
-    )
-    (fp_text value Rxtal (at 2.725 -0.5) (layer B.SilkS)
+    (fp_text reference R4 (at 2.7 3.525) (layer B.SilkS)
+      (effects (font (size 0.8 0.8) (thickness 0.15)) (justify mirror))
+    )
+    (fp_text value Rxtal (at 2.7 0.985) (layer B.SilkS)
       (effects (font (size 0.8 0.8) (thickness 0.15)) (justify mirror))
     )
@@
       (net 27 "Net-(TP8-Pad1)"))
   )
+  (gr_text "ЕС1832\n17072019а0" (at 123.19 62.865 90) (layer F.SilkS)
+    (effects (font (size 0.8 0.8) (thickness 0.15)))
+  )
+  (gr_text "ЕС1832\nТерминален блок\nПроектирано и изработено\nв Република България" (at 132.08 79.375) (layer B.SilkS)
+    (effects (font (size 0.7 0.7) (thickness 0.13)) (justify mirror))
+  )
   (gr_text x2 (at 145.415 60.96) (layer F.SilkS)

Commit message: Improve insignia
Other:
- board text added: "ЕС1832 Терминален възел (ъгъл) Проектирано и изработено в Република България"
- board text removed: "ЕС1832 Терминален блок Проектирано и изработено в Република България"
Changed lines of the file:
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@@
   (page A4)
   (layers
-    (0 F.Cu signal)
-    (31 B.Cu signal)
+    (0 F.Cu signal hide)
+    (31 B.Cu signal hide)
     (32 B.Adhes user)
     (33 F.Adhes user)
@@
     (solder_mask_min_width 0.25)
     (aux_axis_origin 0 0)
-    (visible_elements 7FFFF7FF)
+    (visible_elements 7FFF77FF)
     (pcbplotparams
       (layerselection 0x010fc_ffffffff)
@@
     (tags "resistor handsolder")
     (attr smd)
-    (fp_text reference R4 (at 2.7 3.525) (layer B.SilkS)
-      (effects (font (size 0.8 0.8) (thickness 0.15)) (justify mirror))
-    )
-    (fp_text value Rxtal (at 2.7 0.985) (layer B.SilkS)
+    (fp_text reference R4 (at 1.43 -5.365) (layer B.SilkS)
+      (effects (font (size 0.8 0.8) (thickness 0.15)) (justify mirror))
+    )
+    (fp_text value Rxtal (at 1.43 -2.825) (layer B.SilkS)
       (effects (font (size 0.8 0.8) (thickness 0.15)) (justify mirror))
     )
@@
     (effects (font (size 0.8 0.8) (thickness 0.15)))
   )
-  (gr_text "ЕС1832\nТерминален блок\nПроектирано и изработено\nв Република България" (at 132.08 79.375) (layer B.SilkS)
-    (effects (font (size 0.7 0.7) (thickness 0.13)) (justify mirror))
+  (gr_text "ЕС1832\nТерминален възел (ъгъл)\nПроектирано и изработено\nв Република България" (at 139.065 79.375) (layer B.SilkS)
+    (effects (font (size 0.7 0.7) (thickness 0.13)) (justify left mirror))
   )
   (gr_text x2 (at 145.415 60.96) (layer F.SilkS)
